File: linkup-recreate/pcbs/link-up-serial/link-up-serial/link-up-serial.sch (KiCad schematic (older format))
At the start: 6 parts

Commit message: Updates
Parts:
- added U?: 1489, symbol ajm:1489
- added U?: DS3691, symbol ajm:DS3691
- added U?: ICL7660, symbol Regulator_SwitchedCapacitor:ICL7660
Connections:
- net ORANGE is gone; now on net GND: J?.3 (Pin_3)
- net YELLOW is gone; now on net GND: J?.4 (Pin_4)
- net BLUE: now also U?.1 (IN_A)
- net BROWN: now also U?.15 (OUT_A)
- net GND: now also U?.3 (GND), U?.5 (GND), U?.7 (GND)
- net GREEN: now also U?.4 (IN_B)
- net SD1: now also U?.14
- net Vdd: now also U?.1 (VCC), U?.14 (VCC), U?.8 (V+)
- net CTS_Y: now reaches U?.12
- net CTS_Y: now also U?.13 (IN_D)
- net RXD_X: now reaches U?.16
- net RXD_X: now also U?.10 (IN_C)
- net RTS_X: now reaches U?.15
- net RTS_X: now also U?.6 (OUT_B)
- net TXD_X: now reaches U?.17
- net TXD_X: now also U?.3 (OUT_A)
- new net -5V: U?.5 (VOUT), U?.8 (VEE)
- new net CTS_X: U?.11 (OUT_D), U?.2 (IN_A)
Other:
- note added: "25 pin D type\n\n2: BLUE\n3: RED\n4: GREEN\n5: BROWN\n6: Connected to 20\n7: YELLOW\n20: Connected to 6\n\nORANGE: n.c. (GND)\n"
- note added: "TXD\nRXD\nRTS\nCTS\nDSR\nGND\nDTR"
- note removed: "25 pin D type\n\n2: BLUE\n3: RED\n4: GREEN\n5: BROWN\n6: Connected to 20\n7: YELLOW\n20: onnected to 6\n\nORANGE: n.c.\n"
Changed lines of the file:
@@
 Wire Wire Line
 	2700 2425 2750 2425
-Text GLabel 8625 2425 0    50   Input ~ 0
+Text GLabel 7875 2425 0    50   Input ~ 0
 BROWN
-Text GLabel 8625 2525 0    50   Input ~ 0
+Text GLabel 7875 2525 0    50   Input ~ 0
 RED
-Text GLabel 8625 2625 0    50   Input ~ 0
+Text GLabel 7875 2625 0    50   Input ~ 0
 ORANGE
-Text GLabel 8625 2725 0    50   Input ~ 0
+Text GLabel 7875 2725 0    50   Input ~ 0
 YELLOW
-Text GLabel 8625 2825 0    50   Input ~ 0
+Text GLabel 7875 2825 0    50   Input ~ 0
 GREEN
-Text GLabel 8625 2925 0    50   Input ~ 0
+Text GLabel 7875 2925 0    50   Input ~ 0
 BLUE
 $Comp
@@
 $EndComp
 Wire Wire Line
-	8975 2425 8625 2425
-Wire Wire Line
-	8625 2525 8975 2525
-Wire Wire Line
-	8975 2625 8625 2625
-Wire Wire Line
-	8625 2725 8975 2725
-Wire Wire Line
-	8625 2825 8975 2825
-Wire Wire Line
-	8625 2925 8975 2925
+	8975 2425 7875 2425
+Wire Wire Line
+	7875 2525 8975 2525
+Wire Wire Line
+	8975 2625 8250 2625
+Wire Wire Line
+	7875 2725 8500 2725
+Wire Wire Line
+	7875 2825 8975 2825
+Wire Wire Line
+	7875 2925 8975 2925
 Text Notes 9050 4175 0    50   ~ 0
-25 pin D type\n\n2: BLUE\n3: RED\n4: GREEN\n5: BROWN\n6: Connected to 20\n7: YELLOW\n20: onnected to 6\n\nORANGE: n.c.\n
+25 pin D type\n\n2: BLUE\n3: RED\n4: GREEN\n5: BROWN\n6: Connected to 20\n7: YELLOW\n20: Connected to 6\n\nORANGE: n.c. (GND)\n
 Wire Wire Line
 	4075 3275 4450 3275
@@
 	4925 3150 4450 3150
 Connection ~ 4450 3150
+$Comp
+L ajm:1489 U?
+U 1 1 6371CD69
+P 2050 4400
+F 0 "U?" H 2550 4565 50  0000 C CNN
+F 1 "1489" H 2550 4474 50  0000 C CNN
+F 2 "" H 2050 4400 50  0001 C CNN
+F 3 "" H 2050 4400 50  0001 C CNN
+	1    2050 4400
+	1    0    0    -1
+$EndComp
+$Comp
+L ajm:DS3691 U?
+U 1 1 6371DF57
+P 4025 5800
+F 0 "U?" H 4475 5965 50  0000 C CNN
+F 1 "DS3691" H 4475 5874 50  0000 C CNN
+F 2 "" H 4025 5800 50  0001 C CNN
+F 3 "" H 4025 5800 50  0001 C CNN
+	1    4025 5800
+	1    0    0    -1
+$EndComp
+$Comp
+L Regulator_SwitchedCapacitor:ICL7660 U?
+U 1 1 6371F6A3
+P 4225 1450
+F 0 "U?" H 4225 2017 50  0000 C CNN
+F 1 "ICL7660" H 4225 1926 50  0000 C CNN
+F 2 "" H 4325 1350 50  0001 C CNN
+F 3 "http://datasheets.maximintegrated.com/en/ds/ICL7660-MAX1044.pdf" H 4325 1350 50  0001 C CNN
+	1    4225 1450
+	1    0    0    -1
+$EndComp
+Text GLabel 3600 1150 0    50   Input ~ 0
+SVCC
+Wire Wire Line
+	3600 1150 3825 1150
+$Comp
+L power:GND #PWR?
+U 1 1 63721337
+P 4225 2050
+AR Path="/6104FF77/63721337" Ref="#PWR?"  Part="1"
+AR Path="/63721337" Ref="#PWR?"  Part="1"
+AR Path="/636FE579/63721337" Ref="#PWR?"  Part="1"
+F 0 "#PWR?" H 4225 1800 50  0001 C CNN
+F 1 "GND" H 4225 1875 50  0000 C CNN
+F 2 "" H 4225 2050 50  0001 C CNN
+F 3 "" H 4225 2050 50  0001 C CNN
+	1    4225 2050
+	1    0    0    -1
+$EndComp
+Wire Wire Line
+	4225 2050 4225 1950
+$Comp
+L power:-5V #PWR?
+U 1 1 63721F90
+P 5525 1225
+F 0 "#PWR?" H 5525 1325 50  0001 C CNN
+F 1 "-5V" H 5540 1398 50  0000 C CNN
+F 2 "" H 5525 1225 50  0001 C CNN
+F 3 "" H 5525 1225 50  0001 C CNN
+	1    5525 1225
+	-1   0    0    1
+$EndComp
+$Comp
+L power:-5V #PWR?
+U 1 1 63722CFC
+P 3650 6825
+F 0 "#PWR?" H 3650 6925 50  0001 C CNN
+F 1 "-5V" H 3665 6998 50  0000 C CNN
+F 2 "" H 3650 6825 50  0001 C CNN
+F 3 "" H 3650 6825 50  0001 C CNN
+	1    3650 6825
+	-1   0    0    1
+$EndComp
+Wire Wire Line
+	3925 6600 3650 6600
+Wire Wire Line
+	3650 6600 3650 6825
+Wire Wire Line
+	5525 1150 5525 1225
+Wire Wire Line
+	4625 1150 5525 1150
+Wire Wire Line
+	3925 5900 3650 5900
+$Comp
+L power:GND #PWR?
+U 1 1 63725A73
+P 3150 6450
+F 0 "#PWR?" H 3150 6200 50  0001 C CNN
+F 1 "GND" H 3155 6277 50  0000 C CNN
+F 2 "" H 3150 6450 50  0001 C CNN
+F 3 "" H 3150 6450 50  0001 C CNN
+	1    3150 6450
+	1    0    0    -1
+$EndComp
+Wire Wire Line
+	3925 6300 3150 6300
+Wire Wire Line
+	3150 6300 3150 6450
+Text GLabel 5300 6000 2    50   Input ~ 0
+BROWN
+Wire Wire Line
+	5300 6000 5025 6000
+Text GLabel 4925 3600 0    50   Input ~ 0
+TXD_X
+Text GLabel 2100 4700 0    50   Input ~ 0
+TXD_X
+$Comp
+L power:GND #PWR?
+U 1 1 63727763
+P 1875 5250
+F 0 "#PWR?" H 1875 5000 50  0001 C CNN
+F 1 "GND" H 1880 5077 50  0000 C CNN
+F 2 "" H 1875 5250 50  0001 C CNN
+F 3 "" H 1875 5250 50  0001 C CNN
+	1    1875 5250
+	1    0    0    -1
+$EndComp
+Wire Wire Line
+	2100 5100 1875 5100
+Wire Wire Line
+	1875 5100 1875 5250
+Text GLabel 3650 5900 0    50   Input ~ 0
+SVCC
+Text GLabel 3225 4500 2    50   Input ~ 0
+SVCC
+Wire Wire Line
+	3000 4500 3225 4500
+Text GLabel 2100 4500 0    50   Input ~ 0
+BLUE
+Text Notes 8775 4000 0    50   ~ 0
+TXD\nRXD\nRTS\nCTS\nDSR\nGND\nDTR
+$Comp
+L power:GND #PWR?
+U 1 1 6372AA19
+P 8250 3125
+F 0 "#PWR?" H 8250 2875 50  0001 C CNN
+F 1 "GND" H 8255 2952 50  0000 C CNN
+F 2 "" H 8250 3125 50  0001 C CNN
+F 3 "" H 8250 3125 50  0001 C CNN
+	1    8250 3125
+	1    0    0    -1
+$EndComp
+Wire Wire Line
+	8250 3125 8250 2625
+Connection ~ 8250 2625
+Wire Wire Line
+	8250 2625 7875 2625
+$Comp
+L power:GND #PWR?
+U 1 1 6372B87A
+P 8500 3125
+F 0 "#PWR?" H 8500 2875 50  0001 C CNN
+F 1 "GND" H 8505 2952 50  0000 C CNN
+F 2 "" H 8500 3125 50  0001 C CNN
+F 3 "" H 8500 3125 50  0001 C CNN
+	1    8500 3125
+	1    0    0    -1
+$EndComp
+Wire Wire Line
+	8500 3125 8500 2725
+Connection ~ 8500 2725
+Wire Wire Line
+	8500 2725 8975 2725
+Text GLabel 4075 3375 2    50   Input ~ 0
+RXD_X
+Text GLabel 3000 4900 2    50   Input ~ 0
+RXD_X
+Text GLabel 2100 4800 0    50   Input ~ 0
+GREEN
+Text GLabel 2100 5000 0    50   Input ~ 0
+RTS_X
+Text GLabel 4925 3500 0    50   Input ~ 0
+RTS_X
+Text GLabel 4075 3475 2    50   Input ~ 0
+SD1
+Text GLabel 4075 3575 2    50   Input ~ 0
+CTS_Y
+Text GLabel 3000 4800 2    50   Input ~ 0
+CTS_X
+Text GLabel 3925 6000 0    50   Input ~ 0
+CTS_X
+Text GLabel 3000 4600 2    50   Input ~ 0
+CTS_Y
 $EndSCHEMATC

Commit message: Updates
Connections:
- net RED: now also U?.10 (OUT_D)
- net RXD_X: now also U?.7 (IN_D), U?.8 (OUT_C); no longer U?.10 (IN_C), U?.16
- new net RXD_Y: U?.10 (IN_C), U?.16
Changed lines of the file:
@@
 $Descr A4 11693 8268
 encoding utf-8
-Sheet 1 2
+Sheet 1 1
 Title ""
 Date ""
@@
 Comment4 ""
 $EndDescr
-$Sheet
-S 8175 1150 1050 550
-U 636FE579
-F0 "Sheet636FE578" 50
-F1 "pp.sch" 50
-$EndSheet
 Text GLabel 1475 1775 0    50   Input ~ 0
 SD1
@@
 	8500 2725 8975 2725
 Text GLabel 4075 3375 2    50   Input ~ 0
-RXD_X
+RXD_Y
 Text GLabel 3000 4900 2    50   Input ~ 0
-RXD_X
+RXD_Y
 Text GLabel 2100 4800 0    50   Input ~ 0
 GREEN
@@
 Text GLabel 3000 4600 2    50   Input ~ 0
 CTS_Y
+Text GLabel 3000 5100 2    50   Input ~ 0
+RXD_X
+Text GLabel 3925 6500 0    50   Input ~ 0
+RXD_X
+Text GLabel 5025 6500 2    50   Input ~ 0
+RED
 $EndSCHEMATC

Commit message: Updates
Parts:
- added R?: R_Small, symbol Device:R_Small
Connections:
- net CTS_Y: now also R?.2
- net Vdd: now also R?.1
Changed lines of the file:
@@
 Text GLabel 3650 5900 0    50   Input ~ 0
 SVCC
-Text GLabel 3225 4500 2    50   Input ~ 0
+Text GLabel 3925 4500 2    50   Input ~ 0
 SVCC
-Wire Wire Line
-	3000 4500 3225 4500
 Text GLabel 2100 4500 0    50   Input ~ 0
 BLUE
@@
 Text GLabel 3925 6000 0    50   Input ~ 0
 CTS_X
-Text GLabel 3000 4600 2    50   Input ~ 0
+Text GLabel 3925 4600 2    50   Input ~ 0
 CTS_Y
 Text GLabel 3000 5100 2    50   Input ~ 0
@@
 Text GLabel 5025 6500 2    50   Input ~ 0
 RED
+Wire Wire Line
+	3000 4600 3675 4600
+Wire Wire Line
+	3000 4500 3925 4500
+$Comp
+L Device:R_Small R?
+U 1 1 637324DD
+P 3675 4275
+F 0 "R?" H 3734 4321 50  0000 L CNN
+F 1 "R_Small" H 3734 4230 50  0000 L CNN
+F 2 "" H 3675 4275 50  0001 C CNN
+F 3 "~" H 3675 4275 50  0001 C CNN
+	1    3675 4275
+	1    0    0    -1
+$EndComp
+Text GLabel 3575 4000 0    50   Input ~ 0
+SVCC
+Wire Wire Line
+	3575 4000 3675 4000
+Wire Wire Line
+	3675 4000 3675 4175
+Wire Wire Line
+	3675 4375 3675 4600
+Connection ~ 3675 4600
+Wire Wire Line
+	3675 4600 3925 4600
 $EndSCHEMATC

Commit message: Updates
Parts:
- added C? (x2): 10uF 16V, symbol Device:C_Small
- added C? (x2): 20pF - 10nF, symbol Device:C_Small
- added C?: 100nF?, symbol Device:C_Small
- added R?: 47k, symbol Device:R_Small
Connections:
- net -5V: now also C?.1
- net BROWN: now also C?.2
- net GND: now also C?.2, C?.2, R?.2
- net RED: now also C?.1
- net SMR: now also U?.2, R?.1
- net at U?.6: now also C?.1
- net at U?.16 (RTC_A): now also C?.1
- net at U?.9 (RTC_D): now also C?.2
- net at U?.2 (CAP+): now also C?.1
- net at U?.4 (CAP-): now also C?.2
Changed lines of the file:
@@
 L power:-5V #PWR?
 U 1 1 63721F90
-P 5525 1225
-F 0 "#PWR?" H 5525 1325 50  0001 C CNN
-F 1 "-5V" H 5540 1398 50  0000 C CNN
-F 2 "" H 5525 1225 50  0001 C CNN
-F 3 "" H 5525 1225 50  0001 C CNN
-	1    5525 1225
+P 6300 1225
+F 0 "#PWR?" H 6300 1325 50  0001 C CNN
+F 1 "-5V" H 6315 1398 50  0000 C CNN
+F 2 "" H 6300 1225 50  0001 C CNN
+F 3 "" H 6300 1225 50  0001 C CNN
+	1    6300 1225
 	-1   0    0    1
 $EndComp
@@
 	3650 6600 3650 6825
 Wire Wire Line
-	5525 1150 5525 1225
-Wire Wire Line
-	4625 1150 5525 1150
+	6300 1150 6300 1225
+Wire Wire Line
+	4625 1150 5775 1150
 Wire Wire Line
 	3925 5900 3650 5900
@@
 BROWN
 Wire Wire Line
-	5300 6000 5025 6000
+	5300 6000 5200 6000
 Text GLabel 4925 3600 0    50   Input ~ 0
 TXD_X
@@
 Text GLabel 3925 6500 0    50   Input ~ 0
 RXD_X
-Text GLabel 5025 6500 2    50   Input ~ 0
+Text GLabel 5475 6500 2    50   Input ~ 0
 RED
 Wire Wire Line
@@
 Wire Wire Line
 	3675 4600 3925 4600
+$Comp
+L Device:C_Small C?
+U 1 1 637349F7
+P 5000 1525
+F 0 "C?" H 5092 1571 50  0000 L CNN
+F 1 "10uF 16V" H 5092 1480 50  0000 L CNN
+F 2 "" H 5000 1525 50  0001 C CNN
+F 3 "~" H 5000 1525 50  0001 C CNN
+	1    5000 1525
+	1    0    0    -1
+$EndComp
+Wire Wire Line
+	4625 1350 5000 1350
+Wire Wire Line
+	5000 1350 5000 1425
+Wire Wire Line
+	4625 1750 5000 1750
+Wire Wire Line
+	5000 1750 5000 1625
+$Comp
+L Device:C_Small C?
+U 1 1 63738020
+P 5775 1500
+F 0 "C?" H 5867 1546 50  0000 L CNN
+F 1 "10uF 16V" H 5867 1455 50  0000 L CNN
+F 2 "" H 5775 1500 50  0001 C CNN
+F 3 "~" H 5775 1500 50  0001 C CNN
+	1    5775 1500
+	1    0    0    -1
+$EndComp
+Wire Wire Line
+	5775 1400 5775 1150
+Connection ~ 5775 1150
+Wire Wire Line
+	5775 1150 6300 1150
+$Comp
+L power:GND #PWR?
+U 1 1 637395A7
+P 5775 1700
+F 0 "#PWR?" H 5775 1450 50  0001 C CNN
+F 1 "GND" H 5780 1527 50  0000 C CNN
+F 2 "" H 5775 1700 50  0001 C CNN
+F 3 "" H 5775 1700 50  0001 C CNN
+	1    5775 1700
+	1    0    0    -1
+$EndComp
+Wire Wire Line
+	5775 1600 5775 1700
+$Comp
+L Device:C_Small C?
+U 1 1 6373AE6E
+P 5625 5725
+F 0 "C?" H 5717 5771 50  0000 L CNN
+F 1 "20pF - 10nF" H 5717 5680 50  0000 L CNN
+F 2 "" H 5625 5725 50  0001 C CNN
+F 3 "~" H 5625 5725 50  0001 C CNN
+	1    5625 5725
+	1    0    0    -1
+$EndComp
+Wire Wire Line
+	5025 5900 5100 5900
+Wire Wire Line
+	5100 5900 5100 5575
+Wire Wire Line
+	5100 5575 5625 5575
+Wire Wire Line
+	5625 5575 5625 5625
+Wire Wire Line
+	5625 5825 5200 5825
+Wire Wire Line
+	5200 5825 5200 6000
+Connection ~ 5200 6000
+Wire Wire Line
+	5200 6000 5025 6000
+Wire Wire Line
+	5475 6500 5350 6500
+$Comp
+L Device:C_Small C?
+U 1 1 6373EC72
+P 5350 6700
+F 0 "C?" H 5442 6746 50  0000 L CNN
+F 1 "20pF - 10nF" H 5442 6655 50  0000 L CNN
+F 2 "" H 5350 6700 50  0001 C CNN
+F 3 "~" H 5350 6700 50  0001 C CNN
+	1    5350 6700
+	1    0    0    -1
+$EndComp
+Wire Wire Line
+	5350 6600 5350 6500
+Connection ~ 5350 6500
+Wire Wire Line
+	5350 6500 5025 6500
+Wire Wire Line
+	5350 6800 5350 6875
+Wire Wire Line
+	5350 6875 5100 6875
+Wire Wire Line
+	5100 6875 5100 6600
+Wire Wire Line
+	5100 6600 5025 6600
+$Comp
+L Device:C_Small C?
+U 1 1 637424F4
+P 2550 3675
+F 0 "C?" H 2642 3721 50  0000 L CNN
+F 1 "100nF?" H 2642 3630 50  0000 L CNN
+F 2 "" H 2550 3675 50  0001 C CNN
+F 3 "~" H 2550 3675 50  0001 C CNN
+	1    2550 3675
+	1    0    0    -1
+$EndComp
+Wire Wire Line
+	2550 3575 2550 3475
+Wire Wire Line
+	2550 3475 3075 3475
+$Comp
+L power:GND #PWR?
+U 1 1 63745654
+P 2550 3850
+F 0 "#PWR?" H 2550 3600 50  0001 C CNN
+F 1 "GND" H 2555 3677 50  0000 C CNN
+F 2 "" H 2550 3850 50  0001 C CNN
+F 3 "" H 2550 3850 50  0001 C CNN
+	1    2550 3850
+	1    0    0    -1
+$EndComp
+Wire Wire Line
+	2550 3850 2550 3775
+Text GLabel 2125 3275 0    50   Input ~ 0
+SMR
+Wire Wire Line
+	2125 3275 2200 3275
+$Comp
+L Device:R_Small R?
+U 1 1 637491DA
+P 2200 3500
+F 0 "R?" H 2259 3546 50  0000 L CNN
+F 1 "47k" H 2259 3455 50  0000 L CNN
+F 2 "" H 2200 3500 50  0001 C CNN
+F 3 "~" H 2200 3500 50  0001 C CNN
+	1    2200 3500
+	1    0    0    -1
+$EndComp
+$Comp
+L power:GND #PWR?
+U 1 1 63749883
+P 2200 3875
+F 0 "#PWR?" H 2200 3625 50  0001 C CNN
+F 1 "GND" H 2205 3702 50  0000 C CNN
+F 2 "" H 2200 3875 50  0001 C CNN
+F 3 "" H 2200 3875 50  0001 C CNN
+	1    2200 3875
+	1    0    0    -1
+$EndComp
+Wire Wire Line
+	2200 3875 2200 3600
+Wire Wire Line
+	2200 3400 2200 3275
+Connection ~ 2200 3275
+Wire Wire Line
+	2200 3275 3075 3275
 $EndSCHEMATC

Commit message: Updates
Parts:
- added R?: 10k, symbol Device:R_Small
- added R?: 47k, symbol Device:R_Small
- R?: value R_Small -> 10k
Connections:
- net GND: now also R?.2
- net RXD_Y: now also R?.2
- net SD0: now also U?.8, R?.1
- net SD4: now also U?.4
- net Vdd: now also R?.1
Other:
- moved on the sheet: C?, R?, U?

Commit message: Updates
Parts:
- added R?: 47k, symbol Device:R_Small
Connections:
- net GND: now also U?.11, U?.13, R?.2
- net SD2: now also U?.5
- net SD3: now also U?.3
- net SD4: now also R?.1
- net SS: now also R?.2, U?.1 (~EN)
- net Vdd: no longer R?.2, U?.1 (~EN)
Other:
- moved on the sheet: R?
Changed lines of the file:
@@
 	1    0    0    -1
 $EndComp
-Text GLabel 2550 3125 0    50   Input ~ 0
-SVCC
-Wire Wire Line
-	2550 3125 2700 3125
+Text GLabel 1725 3125 0    50   Input ~ 0
+SS
+Wire Wire Line
+	1725 3125 2700 3125
 Wire Wire Line
 	2700 2875 2700 3125
@@
 Wire Wire Line
 	2550 3925 2550 3850
-Text GLabel 2125 3275 0    50   Input ~ 0
+Text GLabel 1300 3275 0    50   Input ~ 0
 SMR
 Wire Wire Line
-	2125 3275 2200 3275
+	1300 3275 1375 3275
 $Comp
 L Device:R_Small R?
 U 1 1 637491DA
-P 2200 3500
-F 0 "R?" H 2259 3546 50  0000 L CNN
-F 1 "47k" H 2259 3455 50  0000 L CNN
-F 2 "" H 2200 3500 50  0001 C CNN
-F 3 "~" H 2200 3500 50  0001 C CNN
-	1    2200 3500
+P 1375 3500
+F 0 "R?" H 1434 3546 50  0000 L CNN
+F 1 "47k" H 1434 3455 50  0000 L CNN
+F 2 "" H 1375 3500 50  0001 C CNN
+F 3 "~" H 1375 3500 50  0001 C CNN
+	1    1375 3500
 	1    0    0    -1
 $EndComp
@@
 L power:GND #PWR?
 U 1 1 63749883
-P 2200 3925
-F 0 "#PWR?" H 2200 3675 50  0001 C CNN
-F 1 "GND" H 2205 3752 50  0000 C CNN
-F 2 "" H 2200 3925 50  0001 C CNN
-F 3 "" H 2200 3925 50  0001 C CNN
-	1    2200 3925
-	1    0    0    -1
-$EndComp
-Wire Wire Line
-	2200 3925 2200 3600
-Wire Wire Line
-	2200 3400 2200 3275
-Connection ~ 2200 3275
-Wire Wire Line
-	2200 3275 3075 3275
-Text GLabel 2950 3375 0    50   Input ~ 0
+P 1375 3925
+F 0 "#PWR?" H 1375 3675 50  0001 C CNN
+F 1 "GND" H 1380 3752 50  0000 C CNN
+F 2 "" H 1375 3925 50  0001 C CNN
+F 3 "" H 1375 3925 50  0001 C CNN
+	1    1375 3925
+	1    0    0    -1
+$EndComp
+Wire Wire Line
+	1375 3925 1375 3600
+Wire Wire Line
+	1375 3400 1375 3275
+Connection ~ 1375 3275
+Wire Wire Line
+	1375 3275 3075 3275
+Text GLabel 1925 3375 0    50   Input ~ 0
 SD4
-Wire Wire Line
-	2950 3375 3075 3375
 $Comp
 L Device:R_Small R?
@@
 	3025 3575 3075 3575
 Connection ~ 3075 3575
+Wire Wire Line
+	1925 3375 2100 3375
+$Comp
+L Device:R_Small R?
+U 1 1 6377586C
+P 2100 3575
+F 0 "R?" H 2159 3621 50  0000 L CNN
+F 1 "47k" H 2159 3530 50  0000 L CNN
+F 2 "" H 2100 3575 50  0001 C CNN
+F 3 "~" H 2100 3575 50  0001 C CNN
+	1    2100 3575
+	1    0    0    -1
+$EndComp
+$Comp
+L power:GND #PWR?
+U 1 1 63775872
+P 2100 3950
+F 0 "#PWR?" H 2100 3700 50  0001 C CNN
+F 1 "GND" H 2105 3777 50  0000 C CNN
+F 2 "" H 2100 3950 50  0001 C CNN
+F 3 "" H 2100 3950 50  0001 C CNN
+	1    2100 3950
+	1    0    0    -1
+$EndComp
+Wire Wire Line
+	2100 3950 2100 3675
+Wire Wire Line
+	2100 3475 2100 3375
+Connection ~ 2100 3375
+Wire Wire Line
+	2100 3375 3075 3375
+Text GLabel 6075 3600 2    50   Input ~ 0
+SD3
+Wire Wire Line
+	6075 3600 5925 3600
+Text GLabel 6075 3500 2    50   Input ~ 0
+SD2
+Wire Wire Line
+	6075 3500 5925 3500
+$Comp
+L power:GND #PWR?
+U 1 1 6377FAA5
+P 4525 3800
+F 0 "#PWR?" H 4525 3550 50  0001 C CNN
+F 1 "GND" H 4530 3627 50  0000 C CNN
+F 2 "" H 4525 3800 50  0001 C CNN
+F 3 "" H 4525 3800 50  0001 C CNN
+	1    4525 3800
+	1    0    0    -1
+$EndComp
+Wire Wire Line
+	4925 3300 4525 3300
+Wire Wire Line
+	4525 3300 4525 3400
+Wire Wire Line
+	4925 3400 4525 3400
+Connection ~ 4525 3400
+Wire Wire Line
+	4525 3400 4525 3800
 $EndSCHEMATC

Commit message: Updates
Connections:
- net GND: now also U?.3 (IN_B), U?.6 (IN_C)
- net Vdd: now also C?.1, U?.6
Changed lines of the file:
@@
 Wire Wire Line
 	2700 3125 3075 3125
-Text GLabel 2750 2425 2    50   Input ~ 0
+Text GLabel 3075 2425 2    50   Input ~ 0
 SVCC
 Wire Wire Line
 	2700 2675 2700 2425
-Wire Wire Line
-	2700 2425 2750 2425
 Text GLabel 7875 2425 0    50   Input ~ 0
 BROWN
@@
 	4425 6775 3650 6775
 Wire Wire Line
-	3650 6775 3650 6925
+	3650 6775 3650 6875
 Text GLabel 5800 6475 2    50   Input ~ 0
 BROWN
@@
 	2550 3650 2550 3475
 Wire Wire Line
-	2550 3475 3075 3475
+	2550 3475 2975 3475
 $Comp
 L power:GND #PWR?
@@
 Wire Wire Line
 	4525 3400 4525 3800
+Wire Wire Line
+	2700 2425 2975 2425
+Wire Wire Line
+	2975 2425 2975 3475
+Connection ~ 2975 2425
+Wire Wire Line
+	2975 2425 3075 2425
+Connection ~ 2975 3475
+Wire Wire Line
+	2975 3475 3075 3475
+Wire Wire Line
+	4425 6575 3650 6575
+Wire Wire Line
+	3650 6575 3650 6775
+Connection ~ 3650 6775
+Wire Wire Line
+	4425 6875 3650 6875
+Connection ~ 3650 6875
+Wire Wire Line
+	3650 6875 3650 6925
 $EndSCHEMATC

Commit message: Updates
Connections:
- net Vdd: now also U?.4 (MODE_SELECT)
Changed lines of the file:
@@
 Wire Wire Line
 	4625 1150 5775 1150
-Wire Wire Line
-	4425 6375 4150 6375
 $Comp
 L power:GND #PWR?
@@
 Wire Wire Line
 	1875 5600 1875 5750
-Text GLabel 4150 6375 0    50   Input ~ 0
+Text GLabel 3600 6375 0    50   Input ~ 0
 SVCC
 Text GLabel 3925 5000 2    50   Input ~ 0
@@
 Wire Wire Line
 	3650 6875 3650 6925
+Wire Wire Line
+	3600 6375 3950 6375
+Wire Wire Line
+	4425 6675 3950 6675
+Wire Wire Line
+	3950 6675 3950 6375
+Connection ~ 3950 6375
+Wire Wire Line
+	3950 6375 4425 6375
 $EndSCHEMATC
