File: linkup-recreate/pcbs/link-up-serial/link-up-serial/link-up-serial.sch (KiCad schematic (older format))
At the start: 19 parts

Commit message: Updates
Parts:
- C1, C4, C5: renamed from C?; footprint (none) -> Capacitor_SMD:C_0805_2012Metric_Pad1.18x1.45mm_HandSolder
- C2, C3: renamed from C?; footprint (none) -> Capacitor_SMD:C_1210_3225Metric_Pad1.33x2.70mm_HandSolder
- J2: renamed from J?; footprint (none) -> Connector_PinHeader_2.54mm:PinHeader_1x06_P2.54mm_Vertical
- R1, R2, R3, R4, R5, R6, R7: renamed from R?; footprint (none) -> Resistor_SMD:R_0805_2012Metric_Pad1.20x1.40mm_HandSolder
- gave numbers to parts that had none: 5

Commit message: Updates
Parts:
- U1: footprint (none) -> Package_DIP:DIP-14_W7.62mm
- U2: footprint (none) -> Package_SO:SOIC-20W_7.5x12.8mm_P1.27mm
- U3: footprint (none) -> Package_SO:SOP-8_5.28x5.23mm_P1.27mm
- U4: footprint (none) -> Package_DIP:DIP-16_W7.62mm
Changed lines of the file:
@@
 F 0 "U2" H 3575 3941 50  0000 C CNN
 F 1 "40244" H 3575 3850 50  0000 C CNN
-F 2 "" H 3575 3375 50  0001 C CNN
+F 2 "Package_SO:SOIC-20W_7.5x12.8mm_P1.27mm" H 3575 3375 50  0001 C CNN
 F 3 "" H 3575 3375 50  0001 C CNN
 	1    3575 3375
@@
 F 0 "U2" H 5375 3075 50  0000 C CNN
 F 1 "40244" H 5425 2975 50  0000 C CNN
-F 2 "" H 5425 3400 50  0001 C CNN
+F 2 "Package_SO:SOIC-20W_7.5x12.8mm_P1.27mm" H 5425 3400 50  0001 C CNN
 F 3 "" H 5425 3400 50  0001 C CNN
 	2    5425 3400
@@
 F 0 "U1" H 2550 5065 50  0000 C CNN
 F 1 "1489" H 2550 4974 50  0000 C CNN
-F 2 "" H 2050 4900 50  0001 C CNN
+F 2 "Package_DIP:DIP-14_W7.62mm" H 2050 4900 50  0001 C CNN
 F 3 "" H 2050 4900 50  0001 C CNN
 	1    2050 4900
@@
 F 0 "U4" H 4975 6440 50  0000 C CNN
 F 1 "DS3691" H 4975 6349 50  0000 C CNN
-F 2 "" H 4525 6275 50  0001 C CNN
+F 2 "Package_DIP:DIP-16_W7.62mm" H 4525 6275 50  0001 C CNN
 F 3 "" H 4525 6275 50  0001 C CNN
 	1    4525 6275
@@
 F 0 "U3" H 4225 2017 50  0000 C CNN
 F 1 "ICL7660" H 4225 1926 50  0000 C CNN
-F 2 "" H 4325 1350 50  0001 C CNN
+F 2 "Package_SO:SOP-8_5.28x5.23mm_P1.27mm" H 4325 1350 50  0001 C CNN
 F 3 "http://datasheets.maximintegrated.com/en/ds/ICL7660-MAX1044.pdf" H 4325 1350 50  0001 C CNN
 	1    4225 1450
