File: linkup-recreate/pcbs/link-up-serial/link-up-serial/link-up-serial.kicad_pcb (KiCad board)
At the start: 2 copper layers, 49.8 x 20.5 mm, 14 parts, among them J1 Conn_02x08_Odd_Even, J2 Conn_01x06_Female

Commit message: Updates
Parts:
- added U1: 1489, Package_DIP:DIP-14_W7.62mm, F.Cu at (130.8, 113.5)
- added U2: 40244, Package_SO:SOIC-20W_7.5x12.8mm_P1.27mm, B.Cu at (105.9, 110.0)
- added U3: ICL7660, Package_SO:SOP-8_5.28x5.23mm_P1.27mm, F.Cu at (107.2, 117.6)
- added U4: DS3691, Package_DIP:DIP-16_W7.62mm, F.Cu at (131.1, 103.4)
- C1, C2, C3, C5, R2, R5, R6, R7: moved to B.Cu
- moved C2 40.7 mm to (104.4, 120.1)
- moved R5 34.6 mm to (129.5, 118.6), turned to 180 degrees
- moved R2 32.2 mm to (116.3, 117.3)
- moved R6 30.2 mm to (129.5, 116.3), turned to 180 degrees
- moved C1 28.0 mm to (120.4, 107.2), turned to 180 degrees
- moved C5 27.8 mm to (129.5, 107.7), turned to 180 degrees
- moved R4 27.8 mm to (106.4, 113.0), turned to 180 degrees
- moved R1 27.2 mm to (106.9, 106.2), turned to 180 degrees
- moved C4 25.5 mm to (104.4, 108.5)
- moved C3 22.9 mm to (109.7, 120.1), turned to 180 degrees
- moved R7 20.7 mm to (125.2, 107.2)
- moved R3 17.8 mm to (106.9, 104.1), turned to 180 degrees
- moved J2 17.6 mm to (98.8, 105.2)
Connections:
- C2 pad 1: (no net) -> Net-(C2-Pad1)
- C2 pad 2: (no net) -> Net-(C2-Pad2)
- C3 pad 1: (no net) -> -5V
- C4 pad 2: (no net) -> Net-(C4-Pad2)
- C5 pad 1: (no net) -> Net-(C5-Pad1)
- J1 pad 13: (no net) -> SD3
- J1 pad 14: (no net) -> SD2
- J1 pad 15: (no net) -> SD1
- J2 pad 5: (no net) -> GREEN
- J2 pad 6: (no net) -> BLUE
- R5 pad 2: (no net) -> CTS_Y
- R6 pad 2: (no net) -> RXD_Y
- R7 pad 2: (no net) -> Net-(R7-Pad2)

Commit message: Updates
Parts:
- R7: moved to F.Cu
- moved R7 22.8 mm to (102.5, 106.0), turned to 180 degrees
- moved C5 0.92 mm to (129.8, 108.6)
- moved C1 0.90 mm to (119.5, 107.1)
- moved R3 0.25 mm to (106.9, 103.9)
- moved R6 0.25 mm to (129.5, 116.1)
Routing:
- net RXD_Y: track 0.00 -> 44.4 mm, vias 0 -> 3
- net SD3: track 0.00 -> 40.1 mm, vias 0 -> 3
- net CTS_Y: track 0.00 -> 38.6 mm, vias 0 -> 1
- net BLUE: track 0.00 -> 38.3 mm, vias 0 -> 1
- net SD4: track 0.00 -> 35.6 mm, vias 0 -> 3
- net BROWN: track 0.00 -> 35.0 mm, vias 0 -> 1
- net ORANGE: track 0.00 -> 34.7 mm, vias 0 -> 6
- net GREEN: track 0.00 -> 32.9 mm, vias 0 -> 2
- net SD2: track 0.00 -> 32.4 mm, vias 0 -> 1
- net TXD_X: track 0.00 -> 32.4 mm, vias 0 -> 3
- net SVCC: track 0.00 -> 31.1 mm, vias 0 -> 6
- net SD0: track 0.00 -> 30.4 mm, vias 0 -> 3
- net SD1: track 0.00 -> 28.6 mm, vias 0 -> 3
- net SS: track 0.00 -> 27.4 mm, vias 0 -> 3
- net -5V: track 0.00 -> 25.3 mm, vias 0 -> 4
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- added copper zone on In1.Cu, net ORANGE
- added copper zone on In2.Cu, net SVCC
Other:
- copper layers 2 -> 4
